File: etg-pcb/etg-pcb.kicad_pcb (KiCad board)
At the start: 2 copper layers, 1 part

Commit message: Stuff git commit -m Stuff
Parts:
- added H1: MountingHole_Pad, MountingHole:MountingHole_3.2mm_M3_Pad, F.Cu at (155.0, 93.0)
- moved G*** 53.0 mm to (155.0, 118.0)
Routing:
- added copper zone on B.Cu, net GND
- added copper zone on F.Cu, net GND
Other:
- board outline added: 192 x 56.1 mm
